Commit message: working(bad) control on throttle and stearing, track added but not so good

File: description/msauber.xacro (robot description, xacro)
@@ -1,6 +1,13 @@
 <?xml version="1.0" ?>
-<robot xmlns:xacro="http://www.ros.org/wiki/xacro"  name="car">
-    <xacro:include filename="/home/andreas/dev_ws/src/msauber/description/xacro/variables.xacro" />
-    <xacro:include filename="/home/andreas/dev_ws/src/msauber/description/xacro/mesh.xacro" />
-    <xacro:include filename="/home/andreas/dev_ws/src/msauber/description/xacro/effort_control.xacro" />
+<robot xmlns:xacro="http://www.ros.org/wiki/xacro"  name="sauber">
+    <!-- Package resources -->
+    <xacro:arg name="pkg_share" default="$(find msauber)" />
+    <xacro:property name="pkg_share" value="$(arg pkg_share)"/>
+    <xacro:arg name="robot_name" default="sauber" />
+    <xacro:arg name="robot_skin" default="Red" />
+    <xacro:property name="mesh_dir" value="${pkg_share}/description/meshes"/>
+    <xacro:include filename="${pkg_share}/description/xacro/macros.xacro" />
+    <xacro:include filename="${pkg_share}/description/xacro/core.xacro" />
+    <xacro:include filename="${pkg_share}/description/xacro/sensors.xacro" />
+    <xacro:include filename="${pkg_share}/description/xacro/gazebo_plugins.xacro" />
 </robot>

Commit message: ackerman controller and teleop_twist_keyboard for movements

File: description/msauber.xacro (robot description, xacro)
@@ -10,4 +10,4 @@
     <xacro:include filename="${pkg_share}/description/xacro/core.xacro" />
     <xacro:include filename="${pkg_share}/description/xacro/sensors.xacro" />
-    <xacro:include filename="${pkg_share}/description/xacro/gazebo_plugins.xacro" />
+    <xacro:include filename="${pkg_share}/description/xacro/gazebo_plugins_acker.xacro" />
 </robot>

File: description/xacro/core.xacro (robot description, xacro)
@@ -81,5 +81,5 @@
     <child link="$(arg robot_name)_left_steering_hinge" />
     <axis xyz="-1 0 0" />
-    <limit lower="-1.0" upper="1.0" effort="10" velocity="100" />
+    <limit lower="-0.4" upper="0.4" effort="10" velocity="10" />
   </joint>
   <xacro:steering_hinge_transmission name="$(arg robot_name)_left_steering_hinge" />
@@ -99,5 +99,5 @@
     <child link="$(arg robot_name)_right_steering_hinge" />
     <axis xyz="-1 0 0" />
-    <limit lower="-1.0" upper="1.0" effort="10" velocity="100" />
+    <limit lower="-0.4" upper="0.4" effort="10" velocity="10" />
   </joint>
   <xacro:steering_hinge_transmission name="$(arg robot_name)_right_steering_hinge" />
